File: MK_Seq take 3/MK_Seq take 3.kicad_sch (KiCad schematic)
At the start: 122 parts, among them J1 IDC 2x5, Q1 2N3904, Q2 2N3904, Q3 2N3904, Q4 2N3904, Q5 2N3904, Q6 2N3904, Q7 2N3904, Q8 2N3904, Q9 BC548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

Commit message: Working on Seq Rev 3.
Parts:
- added J2: Conn_01x10_Pin, Connector_PinHeader_2.54mm:PinHeader_1x10_P2.54mm_Vertical, symbol Connector:Conn_01x10_Pin
- added J3: Conn_01x10_Pin, Connector_PinSocket_2.54mm:PinSocket_1x10_P2.54mm_Vertical, symbol Connector:Conn_01x10_Pin
- S1: footprint Connector_PinSocket_1.27mm:PinSocket_1x08_P1.27mm_Vertical -> My_Library:Rotary Switch, 1 Pole, 8 Positions
- Step1, Step2, Step3, Step4, Step5, Step6, Step7, Step8: footprint Connector_PinSocket_1.27mm:PinSocket_1x03_P1.27mm_Vertical -> My_Library:Potentiometer_Alpha_RD901F-40-00D_Single_Vertical
Connections:
- net Earth: now also J2.10 (Pin_10), J3.10 (Pin_10)
- net Step1: now also J2.1 (Pin_1), J3.1 (Pin_1)
- net Step2: now also J2.2 (Pin_2), J3.2 (Pin_2)
- net Step3: now also J2.3 (Pin_3), J3.3 (Pin_3)
- net Step4: now also J2.4 (Pin_4), J3.4 (Pin_4)
- net Step5: now also J2.5 (Pin_5), J3.5 (Pin_5)
- net Step6: now also J2.6 (Pin_6), J3.6 (Pin_6)
- net Step7: now also J2.7 (Pin_7), J3.7 (Pin_7)
- net Step8: now also J2.8 (Pin_8), J3.8 (Pin_8)
- net Step9 renamed EOC
- net EOC: now also J2.9 (Pin_9), J3.9 (Pin_9)
Other:
- moved on the sheet: C1, C2, C3, C4, C6, C8, C9, CLK_I1, CLK_O1, CV_O1, D1, D11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
