File: MK_Noise_SH/MK_Noise_SH.kicad_sch (KiCad schematic)
At the start: 40 parts, among them J1 Conn_02x05_Odd_Even, Q1 BC548, U1 TL074

Commit message: 4/26/25
Parts:
- added C12: C_Small, symbol Device:C_Small
- added J2: 3.5mm, symbol My_Symbols:3.5mm_Switched_Mono_Jack
- added R22, R23, R24, R25: R, symbol Device:R
- added RV1: R_Potentiometer, symbol Device:R_Potentiometer
- added U2: TL074, symbol Amplifier_Operational:TL074
Connections:
- new net: R22.2, R23.1, U2.2 (-)
- new net: C12.1, R24.1, U2.3 (+)
- new net: R24.2, RV1.1
- new net: R23.2, R25.1, RV1.2, RV1.3, U2.1
- new net: J2.2 (TN), R25.2
- new net GND: C12.2, J2.1 (S), R22.1
